File: PCB/OrthoTest/OrthoTest.kicad_pcb (KiCad board)
At the start: 2 copper layers, 233.7 x 127.2 mm, 249 parts, among them SW1 SW_Push, SW10 SW_Push, SW11 SW_Push, SW12 SW_Push, SW13 SW_Push, SW14 SW_Push, SW15 SW_Push, SW16 SW_Push, SW17 SW_Push, SW18 SW_Push, SW19 SW_Push, SW2 SW_Push, SW20 SW_Push, SW21 SW_Push, SW22 SW_Push, SW23 SW_Push, SW24 SW_Push, SW25 SW_Push, SW26 SW_Push, SW27 SW_Push, SW28 SW_Push, SW29 SW_Push, SW3 SW_Push, SW30 SW_Push, SW31 SW_Push, SW32 SW_Push, SW33 SW_Push, SW34 SW_Push, SW35 SW_Push, SW36 SW_Push, SW37 SW_Push, SW38 SW_Push, SW39 SW_Push, SW4 SW_Push, SW40 SW_Push, SW41 SW_Push, SW42 SW_Push, SW43 SW_Push, SW44 SW_Push, SW45 SW_Push, SW46 SW_Push, SW47 SW_Push, SW48 SW_Push, SW49 SW_Push, SW5 SW_Push, SW50 SW_Push, SW51 SW_Push, SW52 SW_Push, SW53 SW_Push, SW54 SW_Push, SW55 SW_Push, SW56 SW_Push, SW57 SW_Push, SW58 SW_Push, SW59 SW_Push, SW6 SW_Push, SW60 RotaryEncoder_Switch_MP, SW61 RotaryEncoder_Switch_MP, SW7 SW_Push, SW8 SW_Push, SW9 SW_Push

Commit message: added level shifter and finished rerouting
Parts:
- added U5: SN74LVC1T45DCK, Package_TO_SOT_SMD:SOT-363_SC-70-6, B.Cu at (45.7, 59.1)
Connections:
- A1 pad 21: unconnected-(A1-GPIO16-Pad21) -> row4
- A1 pad 22: unconnected-(A1-GPIO17-Pad22) -> row3
- A1 pad 24: unconnected-(A1-GPIO18-Pad24) -> row2
- A1 pad 25: unconnected-(A1-GPIO19-Pad25) -> row1
- A1 pad 26: unconnected-(A1-GPIO20-Pad26) -> row0
- A1 pad 27: row4 -> col4
- A1 pad 29: row3 -> col3
- A1 pad 31: row2 -> col2
- A1 pad 32: row1 -> col1
- A1 pad 34: row0 -> col0
- A1 pad 35: led_data -> led_data_3v3
- LED1 pad 3: led_data -> led_data_5v
Routing:
- net +3V3: track 0.00 -> 145.8 mm, vias 0 -> 1
- net col5: track 97.6 -> 201.4 mm
- net col4: track 89.5 -> 149.8 mm
- net col3: track 88.9 -> 135.8 mm
- net col2: track 87.0 -> 121.8 mm
- net col1: track 86.9 -> 105.3 mm
- net row0: track 235.4 -> 252.6 mm
- net row1: track 254.8 -> 269.8 mm
- net col0: track 85.0 -> 99.3 mm, vias 0 -> 1
- net row2: track 274.1 -> 287.1 mm
- net led_data: track 12.5 -> 0.00 mm
- net +5V: track 1742.4 -> 1751.3 mm
- net led_data_3v3: track 0.00 -> 8.63 mm
- net row3: track 293.3 -> 301.6 mm
- net led_data_5v: track 0.00 -> 6.47 mm
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